File: hardware/electricity-meter/electricity-meter.kicad_pcb (KiCad board)
At the start: 2 copper layers, 90.2 x 61 mm, 95 parts, among them J1 Conn_01x20_Pin, J2 Conn_01x02_Pin, J3 FTDI breakout, J4 Conn_01x20_Pin, J5 ESB228110100Z, J6 Conn_01x08, J7 RJ45_Shielded, J8 Conn_01x03, J9 Conn_01x03, Q1 BSS138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

Commit message: Update hardware designs
* LED colors
* fix net ties excluded from ibom
Parts:
- D11: value LED -> YELLOW
- D12: value LED -> GREEN
Changed lines of the file:
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@@
         (effects (font (size 1 1) (thickness 0.15)))
     )
-    (fp_text value "LED" (at 1.27 2.96) (layer "F.Fab")
+    (fp_text value "YELLOW" (at 1.27 2.96) (layer "F.Fab")
         (effects (font (size 1 1) (thickness 0.15)))
     )
@@
         (effects (font (size 1 1) (thickness 0.15)))
     )
-    (fp_text value "LED" (at 1.27 2.96) (layer "F.Fab")
-        (effects (font (size 1 1) (thickness 0.15)))
-    )
+    (fp_text value "GREEN" (at 1.27 2.96) (layer "F.Fab")
+        (effects (font (size 1 1) (thickness 0.15)))
+    )
