File: hardware/electricity-meter/modbus.kicad_sch (KiCad schematic)
At the start: 13 parts, among them U4 MAX3485EESA

Commit message: Update documentation
Parts:
- renumbered C7 to C13, C8 to C14, D9 to D13, NT1 to NT5, R17 to R21, R18 to R22, R19 to R23, U4 to U6
Changed lines of the file:
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@@
     (instances
       (project "electricity-meter"
-        (path "/ff3d9e8d-ce05-4912-9770-c80bf98d8dec"
-          (reference "R20") (unit 1)
-        )
         (path "/ff3d9e8d-ce05-4912-9770-c80bf98d8dec/b212e67d-a601-4187-859b-ab25dade484d"
           (reference "R20") (unit 1)
@@
   (symbol (lib_id "power:GND") (at 71.12 91.44 0) (unit 1)
     (in_bom yes) (on_board yes) (dnp no) (fields_autoplaced)
-    (property "Reference" "#PWR033" (at 71.12 97.79 0)
+    (property "Reference" "#PWR053" (at 71.12 97.79 0)
       (effects (font (size 1.27 1.27)) hide)
     )
@@
     (instances
       (project "electricity-meter"
-        (path "/ff3d9e8d-ce05-4912-9770-c80bf98d8dec"
-          (reference "#PWR033") (unit 1)
-        )
         (path "/ff3d9e8d-ce05-4912-9770-c80bf98d8dec/b212e67d-a601-4187-859b-ab25dade484d"
           (reference "#PWR053") (unit 1)
@@
   (symbol (lib_id "Device:R") (at 105.41 72.39 90) (unit 1)
     (in_bom yes) (on_board yes) (dnp no) (fields_autoplaced)
-    (property "Reference" "R17" (at 105.41 67.2297 90)
+    (property "Reference" "R21" (at 105.41 67.2297 90)
       (effects (font (size 1.27 1.27)))
     )
@@
     (instances
       (project "electricity-meter"
-        (path "/ff3d9e8d-ce05-4912-9770-c80bf98d8dec"
-          (reference "R17") (unit 1)
-        )
         (path "/ff3d9e8d-ce05-4912-9770-c80bf98d8dec/b212e67d-a601-4187-859b-ab25dade484d"
           (reference "R21") (unit 1)
@@
   (symbol (lib_id "power:+3V3") (at 88.9 60.96 0) (unit 1)
     (in_bom yes) (on_board yes) (dnp no) (fields_autoplaced)
-    (property "Reference" "#PWR038" (at 88.9 64.77 0)
+    (property "Reference" "#PWR054" (at 88.9 64.77 0)
       (effects (font (size 1.27 1.27)) hide)
     )
@@
     (instances
       (project "electricity-meter"
-        (path "/ff3d9e8d-ce05-4912-9770-c80bf98d8dec"
-          (reference "#PWR038") (unit 1)
-        )
         (path "/ff3d9e8d-ce05-4912-9770-c80bf98d8dec/b212e67d-a601-4187-859b-ab25dade484d"
           (reference "#PWR054") (unit 1)
@@
   (symbol (lib_id "power:GND") (at 50.8 120.65 0) (unit 1)
     (in_bom yes) (on_board yes) (dnp no)
-    (property "Reference" "#PWR040" (at 50.8 127 0)
+    (property "Reference" "#PWR052" (at 50.8 127 0)
       (effects (font (size 1.27 1.27)) hide)
     )
@@
     (instances
       (project "electricity-meter"
-        (path "/ff3d9e8d-ce05-4912-9770-c80bf98d8dec"
-          (reference "#PWR040") (unit 1)
-        )
         (path "/ff3d9e8d-ce05-4912-9770-c80bf98d8dec/b212e67d-a601-4187-859b-ab25dade484d"
           (reference "#PWR052") (unit 1)
@@
   (symbol (lib_id "Diode:SM712_SOT23") (at 138.43 90.17 0) (mirror y) (unit 1)
     (in_bom yes) (on_board yes) (dnp no)
-    (property "Reference" "D9" (at 138.43 84.7811 0)
+    (property "Reference" "D13" (at 138.43 84.7811 0)
       (effects (font (size 1.27 1.27)))
     )
@@
     (instances
       (project "electricity-meter"
-        (path "/ff3d9e8d-ce05-4912-9770-c80bf98d8dec"
-          (reference "D9") (unit 1)
-        )
         (path "/ff3d9e8d-ce05-4912-9770-c80bf98d8dec/b212e67d-a601-4187-859b-ab25dade484d"
           (reference "D13") (unit 1)
@@
   (symbol (lib_id "Device:C") (at 50.8 114.3 0) (unit 1)
     (in_bom yes) (on_board yes) (dnp no)
-    (property "Reference" "C8" (at 53.721 113.1316 0)
+    (property "Reference" "C14" (at 53.721 113.1316 0)
       (effects (font (size 1.27 1.27)) (justify left))
     )
@@
     (instances
       (project "electricity-meter"
-        (path "/ff3d9e8d-ce05-4912-9770-c80bf98d8dec"
-          (reference "C8") (unit 1)
-        )
         (path "/ff3d9e8d-ce05-4912-9770-c80bf98d8dec/b212e67d-a601-4187-859b-ab25dade484d"
           (reference "C14") (unit 1)
@@
   (symbol (lib_id "Interface_UART:MAX3485") (at 88.9 74.93 0) (unit 1)
     (in_bom yes) (on_board yes) (dnp no) (fields_autoplaced)
-    (property "Reference" "U4" (at 91.0941 60.6257 0)
+    (property "Reference" "U6" (at 91.0941 60.6257 0)
       (effects (font (size 1.27 1.27)) (justify left))
     )
@@
     (instances
       (project "electricity-meter"
-        (path "/ff3d9e8d-ce05-4912-9770-c80bf98d8dec"
-          (reference "U4") (unit 1)
-        )
         (path "/ff3d9e8d-ce05-4912-9770-c80bf98d8dec/b212e67d-a601-4187-859b-ab25dade484d"
           (reference "U6") (unit 1)
@@
   (symbol (lib_id "Device:C") (at 38.1 114.3 0) (unit 1)
     (in_bom yes) (on_board yes) (dnp no)
-    (property "Reference" "C7" (at 41.021 113.1316 0)
+    (property "Reference" "C13" (at 41.021 113.1316 0)
       (effects (font (size 1.27 1.27)) (justify left))
     )
@@
     (instances
       (project "electricity-meter"
-        (path "/ff3d9e8d-ce05-4912-9770-c80bf98d8dec"
-          (reference "C7") (unit 1)
-        )
         (path "/ff3d9e8d-ce05-4912-9770-c80bf98d8dec/b212e67d-a601-4187-859b-ab25dade484d"
           (reference "C13") (unit 1)
@@
   (symbol (lib_id "power:GND") (at 88.9 92.71 0) (unit 1)
     (in_bom yes) (on_board yes) (dnp no) (fields_autoplaced)
-    (property "Reference" "#PWR034" (at 88.9 99.06 0)
+    (property "Reference" "#PWR055" (at 88.9 99.06 0)
       (effects (font (size 1.27 1.27)) hide)
     )
@@
     (instances
       (project "electricity-meter"
-        (path "/ff3d9e8d-ce05-4912-9770-c80bf98d8dec"
-          (reference "#PWR034") (unit 1)
-        )
         (path "/ff3d9e8d-ce05-4912-9770-c80bf98d8dec/b212e67d-a601-4187-859b-ab25dade484d"
           (reference "#PWR055") (unit 1)
@@
   (symbol (lib_id "power:+3V3") (at 50.8 107.95 0) (unit 1)
     (in_bom yes) (on_board yes) (dnp no)
-    (property "Reference" "#PWR039" (at 50.8 111.76 0)
+    (property "Reference" "#PWR051" (at 50.8 111.76 0)
       (effects (font (size 1.27 1.27)) hide)
     )
@@
     (instances
       (project "electricity-meter"
-        (path "/ff3d9e8d-ce05-4912-9770-c80bf98d8dec"
-          (reference "#PWR039") (unit 1)
-        )
         (path "/ff3d9e8d-ce05-4912-9770-c80bf98d8dec/b212e67d-a601-4187-859b-ab25dade484d"
           (reference "#PWR051") (unit 1)
@@
   (symbol (lib_id "Device:R") (at 113.03 76.2 0) (unit 1)
     (in_bom yes) (on_board yes) (dnp no) (fields_autoplaced)
-    (property "Reference" "R19" (at 114.808 74.9879 0)
+    (property "Reference" "R23" (at 114.808 74.9879 0)
       (effects (font (size 1.27 1.27)) (justify left))
     )
@@
     (instances
       (project "electricity-meter"
-        (path "/ff3d9e8d-ce05-4912-9770-c80bf98d8dec"
-          (reference "R19") (unit 1)
-        )
         (path "/ff3d9e8d-ce05-4912-9770-c80bf98d8dec/b212e67d-a601-4187-859b-ab25dade484d"
           (reference "R23") (unit 1)
@@
   (symbol (lib_id "power:GND") (at 138.43 95.25 0) (unit 1)
     (in_bom yes) (on_board yes) (dnp no) (fields_autoplaced)
-    (property "Reference" "#PWR035" (at 138.43 101.6 0)
+    (property "Reference" "#PWR057" (at 138.43 101.6 0)
       (effects (font (size 1.27 1.27)) hide)
     )
@@
     (instances
       (project "electricity-meter"
-        (path "/ff3d9e8d-ce05-4912-9770-c80bf98d8dec"
-          (reference "#PWR035") (unit 1)
-        )
         (path "/ff3d9e8d-ce05-4912-9770-c80bf98d8dec/b212e67d-a601-4187-859b-ab25dade484d"
           (reference "#PWR057") (unit 1)
@@
   (symbol (lib_id "Device:NetTie_2") (at 123.19 80.01 0) (unit 1)
     (in_bom no) (on_board yes) (dnp no) (fields_autoplaced)
-    (property "Reference" "NT1" (at 123.19 81.7301 0)
+    (property "Reference" "NT5" (at 123.19 81.7301 0)
       (effects (font (size 1.27 1.27)))
     )
@@
     (instances
       (project "electricity-meter"
-        (path "/ff3d9e8d-ce05-4912-9770-c80bf98d8dec"
-          (reference "NT1") (unit 1)
-        )
         (path "/ff3d9e8d-ce05-4912-9770-c80bf98d8dec/b212e67d-a601-4187-859b-ab25dade484d"
           (reference "NT5") (unit 1)
@@
   (symbol (lib_id "Device:R") (at 105.41 80.01 90) (unit 1)
     (in_bom yes) (on_board yes) (dnp no) (fields_autoplaced)
-    (property "Reference" "R18" (at 105.41 74.8497 90)
+    (property "Reference" "R22" (at 105.41 74.8497 90)
       (effects (font (size 1.27 1.27)))
     )
@@
     (instances
       (project "electricity-meter"
-        (path "/ff3d9e8d-ce05-4912-9770-c80bf98d8dec"
-          (reference "R18") (unit 1)
-        )
         (path "/ff3d9e8d-ce05-4912-9770-c80bf98d8dec/b212e67d-a601-4187-859b-ab25dade484d"
           (reference "R22") (unit 1)
