File: hardware/electricity-meter/onewire.kicad_sch (KiCad schematic)
At the start: 12 parts, among them J8 Conn_01x03, J9 Conn_01x03, Q1 BSS138

Commit message: Update documentation
Parts:
- renumbered D5 to D15, D5 to D16, NT1 to NT6, NT1 to NT7
Changed lines of the file:
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@@
   (symbol (lib_id "Device:NetTie_2") (at 95.25 30.48 90) (unit 1)
     (in_bom no) (on_board yes) (dnp no) (fields_autoplaced)
-    (property "Reference" "NT1" (at 96.012 29.2679 90)
+    (property "Reference" "NT7" (at 96.012 29.2679 90)
       (effects (font (size 1.27 1.27)) (justify right))
     )
@@
     (instances
       (project "electricity-meter"
-        (path "/ff3d9e8d-ce05-4912-9770-c80bf98d8dec"
-          (reference "NT1") (unit 1)
-        )
         (path "/ff3d9e8d-ce05-4912-9770-c80bf98d8dec/1be1bd7a-4bec-4e66-96e9-7d210635ed68"
           (reference "NT7") (unit 1)
@@
   (symbol (lib_id "Device:NetTie_2") (at 73.66 63.5 0) (unit 1)
     (in_bom no) (on_board yes) (dnp no)
-    (property "Reference" "NT1" (at 73.66 62.23 0)
+    (property "Reference" "NT6" (at 73.66 62.23 0)
       (effects (font (size 1.27 1.27)))
     )
@@
     (instances
       (project "electricity-meter"
-        (path "/ff3d9e8d-ce05-4912-9770-c80bf98d8dec"
-          (reference "NT1") (unit 1)
-        )
         (path "/ff3d9e8d-ce05-4912-9770-c80bf98d8dec/1be1bd7a-4bec-4e66-96e9-7d210635ed68"
           (reference "NT6") (unit 1)
@@
   (symbol (lib_id "Diode:ESD5Zxx") (at 139.7 69.85 270) (unit 1)
     (in_bom yes) (on_board yes) (dnp no) (fields_autoplaced)
-    (property "Reference" "D5" (at 141.732 68.6379 90)
+    (property "Reference" "D15" (at 141.732 68.6379 90)
       (effects (font (size 1.27 1.27)) (justify left))
     )
@@
     (instances
       (project "electricity-meter"
-        (path "/ff3d9e8d-ce05-4912-9770-c80bf98d8dec"
-          (reference "D5") (unit 1)
-        )
         (path "/ff3d9e8d-ce05-4912-9770-c80bf98d8dec/1be1bd7a-4bec-4e66-96e9-7d210635ed68"
           (reference "D15") (unit 1)
@@
   (symbol (lib_id "Diode:ESD5Zxx") (at 228.6 63.5 270) (unit 1)
     (in_bom yes) (on_board yes) (dnp no) (fields_autoplaced)
-    (property "Reference" "D5" (at 230.632 62.2879 90)
+    (property "Reference" "D16" (at 230.632 62.2879 90)
       (effects (font (size 1.27 1.27)) (justify left))
     )
@@
     (instances
       (project "electricity-meter"
-        (path "/ff3d9e8d-ce05-4912-9770-c80bf98d8dec"
-          (reference "D5") (unit 1)
-        )
         (path "/ff3d9e8d-ce05-4912-9770-c80bf98d8dec/1be1bd7a-4bec-4e66-96e9-7d210635ed68"
           (reference "D16") (unit 1)
